Commit message: update

File: URDF/05-sarge5_v1.urdf (robot description, URDF)
Before this commit: robot sarge5_v1, 13 links, 12 joints
Links:
- added link front_left_end_effector; collision sphere radius=0.1; visual sphere radius=0.1
Joints:
- added joint front_left_foot_to_front_left_end_effector: type fixed, parent front_left_foot, child front_left_end_effector, origin xyz=1.02 0 0 rpy=0 0 0
- joint front_left_knee_to_front_left_foot: limit lower=-1.57075 upper=1.57075 effort=1000.0 velocity=10 -> lower=-3.1415 upper=3.1415 effort=1000.0 velocity=10

Commit message: robot standing

File: URDF/05-sarge5_v1.urdf (robot description, URDF)
Before this commit: robot sarge5_v1, 14 links, 13 joints
Links:
- added link back_left_end_effector, mass 3; collision sphere radius=0.1; visual sphere radius=0.1
- added link back_right_end_effector, mass 3; collision sphere radius=0.1; visual sphere radius=0.1
- added link front_right_end_effector, mass 3; collision sphere radius=0.1; visual sphere radius=0.1
- link front_left_end_effector: mass None -> 3
Joints:
- added joint back_left_foot_to_back_left_end_effector: type fixed, parent back_left_foot, child back_left_end_effector, origin xyz=1.02 0 0 rpy=0 0 0
- added joint back_right_foot_to_back_right_end_effector: type fixed, parent back_right_foot, child back_right_end_effector, origin xyz=1.02 0 0 rpy=0 0 0
- added joint front_right_foot_to_front_right_end_effector: type fixed, parent front_right_foot, child front_right_end_effector, origin xyz=1.02 0 0 rpy=0 0 0

Commit message: UPDATE WALKING

File: URDF/05-sarge5_v1.urdf (robot description, URDF)
Before this commit: robot sarge5_v1, 17 links, 16 joints
Links:
- link back_left_end_effector: mass 3 -> 0.1
- link back_left_foot: mass 3 -> 0.1
- link back_left_hip: mass 3 -> 0.1
- link back_left_knee: mass 3 -> 0.1
- link back_right_end_effector: mass 3 -> 0.1
- link back_right_foot: mass 3 -> 0.1
- link back_right_hip: mass 3 -> 0.1
- link back_right_knee: mass 3 -> 0.1
- link base_link: mass 10 -> 1
- link front_left_end_effector: mass 3 -> 0.1
- link front_left_foot: mass 3 -> 0.1
- link front_left_hip: mass 3 -> 0.1
- link front_left_knee: mass 3 -> 0.1
- link front_right_end_effector: mass 3 -> 0.1
- link front_right_foot: mass 3 -> 0.1
- link front_right_hip: mass 3 -> 0.1
- link front_right_knee: mass 3 -> 0.1
